File: kicad-files/OpenHardwareExG_Shield.sch (KiCad schematic (older format))
At the start: 129 parts, among them P11 ARDUINO_SHIELD, U1 ADS1299, U15 TL431BIDBZR, U4 BT1308W-600D, U9 74AUP1G125GW

Commit message: connected DRDY, DOUT, and CS for MASTER and SLAVEs
Parts:
- removed C82: 100nF, SM0603, symbol C
- removed R85: 47, SM0603, symbol R
- removed U9: 74AUP1G125GW, SOT353, symbol 74AUP1G125GW
- added U? (x3): 74LS125, ~, symbol 74LS125
- added U? (x3): 74LS00, ~, symbol 74LS00
- added U? (x3): 74LS02, ~, symbol 74LS02
Connections:
- net labels added: MASTER_DOUT, MASTER_~CS~, MASTER_~DRDY~, SLAVE_~CS~, VCC, ~ENABLED_MISO~, ~MASTER~
- net labels removed: CS_MASTER, CS_SLAVE, DATA_READY
- wire segments 471 -> 500
Other:
- note added: "note: check to see if we can get 3 different footprints of widely available parts"
- note removed: "Allows other SPI devices to drive MISO"

Commit message: add more labels
Connections:
- net labels added: MASTER_AND_MASTER_CS, SLAVE_AND_SLAVE_CS
Changed lines of the file:
@@
 Sheet 1 1
 Title ""
-Date "11 oct 2014"
+Date "18 oct 2014"
 Rev ""
 Comp ""
@@
 	2000 18950 2300 18950
 Connection ~ 2300 18950
+Text Label 29150 8600 0    60   ~ 0
+MASTER_AND_MASTER_CS
+Text Label 29150 9250 0    60   ~ 0
+SLAVE_AND_SLAVE_CS
 $EndSCHEMATC

Commit message: added capacitors for logic chips
Also distinguish ARDUINO_VCC from filtered VCC
Parts:
- added C? (x3): 100nF, SM0603, symbol C
- added C?: 10uF, SM0805, symbol C
- added L?: MH2029-221Y, SM0805, symbol INDUCTOR
Connections:
- net labels added: ARDUINO_VCC
- wire segments 500 -> 642
Other:
- note added: "Buffer"
- note added: "NAND"
- note added: "NOR"
- note added: "capacitors for logic chips"

Commit message: isolated side of ADuM6000 hooked up
Parts:
- added C? (x4): 100nF, SM0603, symbol C
- added C? (x4): 10uF, SM0805, symbol C
- added L? (x2): MH2029-221Y, SM0805, symbol INDUCTOR
- added R?: 0, ~, symbol R
- added R?: NI, ~, symbol R
Connections:
- net labels added: VSEL
- wire segments 642 -> 565
Other:
- note added: "For 5V, connect VIN_ISO to VSEL\nand disconnect VSEL from DGND"
- note added: "Note that bypass capacitors should be\nvery close to the chip and the grounds\nconnectted together with a very low\nimpedence connection\n(wide traces, large vias)"
- note added: "bypass capacitors"
- moved on the sheet: C?, R?, U?

Commit message: non-isolated side of ADuM6000 hooked up
Connections:
- wire segments 565 -> 567
- no-connect marks 11 -> 13
Changed lines of the file:
@@
 Text Notes 18350 7500 0    39   ~ 0
 For 5V, connect VIN_ISO to VSEL\nand disconnect VSEL from DGND
+Wire Wire Line
+	25450 2000 26050 2000
+Wire Wire Line
+	26050 2000 26050 2100
+Connection ~ 26050 2100
+NoConn ~ 25450 1800
+NoConn ~ 25450 1900
 $EndSCHEMATC

Commit message: add test points and NC unused pins
Parts:
- removed P?: CONN_2, symbol CONN_2
- added K?: CONN_3, symbol CONN_3
- added P? (x15): CONN_1, symbol CONN_1
Connections:
- net labels removed: BIASIN, GND_ISO, SRB1, SRB2
- wire segments 567 -> 580
- no-connect marks 13 -> 15
Other:
- note removed: "BIASIN is\ncurrently\nunused"

Commit message: fixed labels and ERC issues
Parts:
- gave numbers to parts that had none: 47
- renumbered C99 to C17, C17 to C18, C18 to C19, C19 to C20, C20 to C21, C21 to C22, C22 to C23, C23 to C24, C24 to C25, C25 to C26, C26 to C27, C27 to C28, C28 to C29, C29 to C30, C30 to C31, C31 to C32, C32 to C33, C101 to C34, C33 to C35, C34 to C36, C35 to C37, C36 to C38, C37 to C39, C38 to C40, C39 to C41, C40 to C42, C60 to C43, C43 to C44, C46 to C45, C47 to C46, C48 to C47, C50 to C48, C51 to C49, C53 to C50, C55 to C51, C49 to C53, C52 to C54, C54 to C55, C64 to C61, C68 to C62, C71 to C63, C75 to C64, D6 to D1, L10 to L6, P11 to P2, R55 to R17, R17 to R18, R18 to R19, R19 to R20, R20 to R21, R21 to R22, R22 to R23, R23 to R24, R24 to R25, R25 to R26, R26 to R27, R27 to R28, R28 to R29, R29 to R30, R30 to R31, R31 to R32, R32 to R33, R56 to R34, R58 to R35, R33 to R36, R66 to R37, R67 to R38, R60 to R39, R62 to R41, R65 to R42, R45 to R46, R78 to R47, R79 to R48, R80 to R49, R84 to R50, U4 to U2, U15 to U3
Connections:
- net labels removed: ADS129x_SCLK, RESET, V_IN
- wire segments 580 -> 579
- no-connect marks 15 -> 29

Commit message: added test points for all I/O to the OpenHardwareExG_Shield
Parts:
- added P1, P11, P12, P13, P14, P17, P18, P2, P29, P3, P30, P31, P32, P33, P34, P35, P36, P37, P38, P4, P46, P47, P48, P49, P5, P50, P51, P52, P53, P54, P55, P6, P7, P8, P9: CONN_1, symbol CONN_1
- renumbered P1 to P10, P2 to P19, P3 to P20, P4 to P21, P5 to P22, P6 to P23, P7 to P24, P8 to P25, P9 to P26, P10 to P27, P11 to P28, P12 to P39, P13 to P40, P14 to P41, P17 to P42, P18 to P43, P19 to P44, P20 to P45
Connections:
- net labels added: ARDUINO_3.3V, ARDUINO_5V, ARDUINO_GND, DGND_ISO
- wire segments 579 -> 617
Other:
- note added: "Test Points"
- moved on the sheet: P39, P40, P41, P42, P43, P44, P45
