File: kicad-files/OpenHardwareExG_Shield_Test_Board.sch (KiCad schematic (older format))
At the start: 86 parts, among them K1 CONN_3, P1 CONN_10X2, P10 CONN_1, P11 CONN_1, P12 CONN_1, P13 CONN_1, P14 CONN_1, P15 CONN_1, P16 CONN_1, P17 CONN_1, P18 CONN_1, P19 CONN_1, P2 ARDUINO_SHIELD, P20 CONN_1, P3 CONN_3X2, P4 CONN_3X2, P5 CONN_4, P6 CONN_1, P7 CONN_1, P8 CONN_1, P9 CONN_1, U4 NI, U5 ADUM6000

Commit message: Test_Board now uses all the test points for I/O to shield
Parts:
- removed C52, C56: NI, ~, symbol C
- removed C69: 10uF, SM0805, symbol C
- removed C70, C71, C72: 100nF, SM0603, symbol C
- removed K1: CONN_3, symbol CONN_3
- removed L7: MH2029-221Y, SM0805, symbol INDUCTOR
- removed P1: CONN_10X2, symbol CONN_10X2
- removed P3, P4: CONN_3X2, symbol CONN_3X2
- removed P5: CONN_4, symbol CONN_4
- removed P?: CONN_1, symbol CONN_1
- removed R43: NI, ~, symbol R
- removed R44, R45: 0, ~, symbol R
- removed U4: NI, symbol LM317_SOT223
- added C1: 10uF, SM0805, symbol C
- added C2, C3, C4: 100nF, SM0603, symbol C
- added D2, D3: LED, LED-0603, symbol LED
- added L1: MH2029-221Y, SM0805, symbol INDUCTOR
- added P2, P21, P22, P23, P24, P25, P26, P27, P28, P29, P3, P30, P31, P32, P33, P34, P35, P36, P37, P38, P39, P4, P40, P41, P42, P43, P44, P45, P46, P47, P48, P49, P5, P50, P51: CONN_1, symbol CONN_1
- added R27, R28: 560, SM0603, symbol R
- added R29, R30: 10k, ~, symbol R
- added SW1: SW_PUSH, ~, symbol SW_PUSH
- added U3: 74HC595PWR, ~, symbol 74HC595PWR
- added U4: 74HC165, symbol 74HC165
- added U5: 74LS125, ~, symbol 74LS125
- added U6: TPS2095D, ~, symbol TPS2095D
- gave numbers to parts that had none: 31
- renumbered C62 to C10, C63 to C11, C64 to C12, C65 to C13, C66 to C14, C67 to C15, C68 to C16, C57 to C5, C58 to C6, C59 to C7, C60 to C8, C61 to C9, L4 to L2, L5 to L3, L6 to L4, L8 to L5, P2 to P1, R35 to R26, R48 to R32, R49 to R33, R50 to R36, U5 to U7
Connections:
- net labels added: 3.3V_BOGUS_ISO, ARDUINO_3.3V, ARDUINO_5V, ARDUINO_GND, DGND_ISO, ENABLE_SHIELD, FAULT_LED, GNDPWR, GND_BOGUS_ISO, GO_BUTTON, SHIELD_3.3V, SHIELD_5V, SHIELD_SHORTED, SHIELD_VCC, SHIFT_CARRY, SHIFT_CARRY_ISO, SHIFT_IN, SHIFT_OUT_RCLK, SHIFT_OUT_SRCLK, SHIFT_OUT_~SRCLR~, SUCCESS_LED, VIN_BOGUS_ISO, ~SEND_TO_GND~_MASTER, ~SEND_TO_GND~_MASTER_ISO
- net labels removed: ADS129x_START_ISO, ADS129x_~PWDN~_ISO, ADS129x_~RESET~_ISO, AGND, DGND, DRIVE_MASTER, DRIVE_MASTER_ISO, SHIFT_OUT_ISO, VSEL
- wire segments 340 -> 372
- no-connect marks 18 -> 19
Other:
- note added: "Fault Indicator"
- note added: "SHIFT"
- note added: "Success Indicator"
- note added: "Test Pogos"
- note removed: "For 5V, connect VIN_ISO to VSEL\nand disconnect VSEL from DGND"
- note removed: "For 5V\n(required by ADS1299)\nuse NCP1117LPST33T3G\nand 10uF capacitors\nand remove 0 Ohm resistor"
- note removed: "Header for isolated analog inputs"
- note removed: "NAND"
- note removed: "NOR"
- note removed: "TODO"
- note removed: "Topside connector"
- note removed: "Underside connector"

Commit message: add pulldown resistors to pogo inputs
Parts:
- added R10, R11, R12, R13, R14, R15, R16, R34, R35, R36, R37, R38, R9: 1M, ~, symbol R
- renumbered R9 to R17, R10 to R18, R11 to R19, R12 to R20, R13 to R21, R14 to R22, R15 to R23, R16 to R24, R17 to R25, R18 to R26, R19 to R27, R20 to R28, R21 to R29, R22 to R30, R23 to R31, R24 to R32, R25 to R33, R26 to R39, R27 to R40, R28 to R41, R29 to R42, R30 to R43, R31 to R44, R32 to R45, R33 to R46, R34 to R47, R35 to R48, R36 to R49
Connections:
- wire segments 372 -> 406
Other:
- moved on the sheet: U1

Commit message: added jumper block for input of calibration signals
Parts:
- added P2: CONN_3X2, symbol CONN_3X2
- added P3: CONN_20X2, symbol CONN_20X2
- added R38: 1M, ~, symbol R
- renumbered P8 to P10, P9 to P11, P10 to P12, P11 to P13, P12 to P14, P13 to P15, P14 to P16, P15 to P17, P16 to P18, P17 to P19, P18 to P20, P19 to P21, P20 to P22, P21 to P23, P22 to P24, P23 to P25, P24 to P26, P25 to P27, P26 to P28, P27 to P29, P28 to P30, P29 to P31, P30 to P32, P31 to P33, P32 to P34, P33 to P35, P34 to P36, P35 to P37, P36 to P38, P37 to P39, P2 to P4, P38 to P40, P39 to P41, P40 to P42, P41 to P43, P42 to P44, P43 to P45, P44 to P46, P45 to P47, P46 to P48, P47 to P49, P3 to P5, P48 to P50, P49 to P51, P50 to P52, P51 to P53, P4 to P6, P5 to P7, P6 to P8, P7 to P9, R38 to R39, R39 to R40, R40 to R41, R41 to R42, R42 to R43, R43 to R44, R44 to R45, R45 to R46, R46 to R47, R47 to R48, R48 to R49, R49 to R50
Connections:
- net labels added: IN1N_LADDER, IN1P_LADDER, IN2N_LADDER, IN2P_LADDER, IN3N_LADDER, IN3P_LADDER, IN4N_LADDER, IN4P_LADDER, IN5N_LADDER, IN5P_LADDER, IN6N_LADDER, IN6P_LADDER, IN7N_LADDER, IN7P_LADDER, IN8N_LADDER, IN8P_LADDER, SHIFT_EXT_CARRY_ISO, SIGNAL_A_LADDER, SIGNAL_B_LADDER
- wire segments 406 -> 451
- no-connect marks 19 -> 22

Commit message: Clarify that all isolation on the test board is actually BOGUS
Connections:
- net labels added: ADS129x_CLK_BOGUS_ISO, ADS129x_DAISY_IN_BOGUS_ISO, ADS129x_DOUT_BOGUS_ISO, ADS129x_GPIO1_BOGUS_ISO, ADS129x_GPIO2_BOGUS_ISO, ADS129x_GPIO3_BOGUS_ISO, ADS129x_GPIO4_BOGUS_ISO, ADS129x_MOSI_BOGUS_ISO, ADS129x_SCLK_BOGUS_ISO, ADS129x_~CS~_BOGUS_ISO, ADS129x_~DRDY~_BOGUS_ISO, DGND_BOGUS_ISO, MASTER_BOGUS_ISO, SHIFT_CARRY_BOGUS_ISO, SHIFT_CLK_BOGUS_ISO, SHIFT_EXT_CARRY_BOGUS_ISO, SHIFT_SH_~LD~_BOGUS_ISO, SIGNAL_A_BOGUS_ISO, SIGNAL_B_BOGUS_ISO, ~SEND_TO_GND~_MASTER_BOGUS_ISO
- net labels removed: 3.3V_ISO, ADS129x_CLK_ISO, ADS129x_DAISY_IN_ISO, ADS129x_DOUT_ISO, ADS129x_GPIO1_ISO, ADS129x_GPIO2_ISO, ADS129x_GPIO3_ISO, ADS129x_GPIO4_ISO, ADS129x_MOSI_ISO, ADS129x_SCLK_ISO, ADS129x_~CS~_ISO, ADS129x_~DRDY~_ISO, DGND_ISO, MASTER_ISO, SHIFT_CARRY_ISO, SHIFT_CLK_ISO, SHIFT_EXT_CARRY_ISO, SHIFT_SH_~LD~_ISO, SIGNAL_A_ISO, SIGNAL_B_ISO, VIN_ISO, ~SEND_TO_GND~_MASTER_ISO
- wire segments 451 -> 549
