File: kicad-files/OpenHardwareExG_Shield_Test_Board.sch (KiCad schematic (older format))
At the start: 136 parts, among them P1 ARDUINO_SHIELD, P10 CONN_1, P11 CONN_1, P12 CONN_1, P13 CONN_1, P14 CONN_1, P15 CONN_1, P16 CONN_1, P17 CONN_1, P18 CONN_1, P19 CONN_1, P2 CONN_3X2, P20 CONN_1, P21 CONN_1, P22 CONN_1, P23 CONN_1, P24 CONN_1, P25 CONN_1, P26 CONN_1, P27 CONN_1, P28 CONN_1, P29 CONN_1, P3 CONN_20X2, P30 CONN_1, P31 CONN_1, P32 CONN_1, P33 CONN_1, P34 CONN_1, P35 CONN_1, P36 CONN_1, P37 CONN_1, P38 CONN_1, P39 CONN_1, P4 CONN_1, P40 CONN_1, P41 CONN_1, P42 CONN_1, P43 CONN_1, P44 CONN_1, P45 CONN_1, P46 CONN_1, P47 CONN_1, P48 CONN_1, P49 CONN_1, P5 CONN_1, P50 CONN_1, P51 CONN_1, P52 CONN_1, P53 CONN_1, P6 CONN_1, P7 CONN_1, P8 CONN_1, P9 CONN_1, SW1 SW_PUSH, U1 74HC165, U2 74HC165, U3 74HC595PWR, U4 74HC165, U5 74LS125, U6 TPS2095D, U7 ADUM6000, U8 SI8661

Commit message: add non-isolated powerlines to test board test signal header
Connections:
- wire segments 549 -> 454
- no-connect marks 22 -> 19

Commit message: add footprints to schematics
Parts:
- P10, P11, P12, P13, P14, P15, P16, P17, P18, P19, P20, P21, P22, P23, P24, P25, P26, P27, P28, P29, P30, P31, P32, P33, P34, P35, P36, P37, P38, P39, P4, P40, P41, P42, P43, P44, P45, P46, P47, P48, P49, P5, P50, P51, P52, P53, P6, P7, P8, P9: footprint (none) -> POGO_PIN_BASE
- P2: footprint (none) -> pin_array_3x2
- P3: footprint (none) -> PIN_ARRAY_20X2
- R1, R17, R18, R19, R2, R20, R21, R22, R23, R24, R25, R26, R27, R28, R29, R3, R30, R31, R32, R33, R4, R43, R44, R5, R6, R7, R8: footprint ~ -> SM0603
- R10, R11, R12, R13, R14, R15, R16, R34, R35, R36, R37, R38, R39, R9: footprint ~ -> SM0805
- SW1: footprint ~ -> smt-tactile-button
- U1, U2, U4: footprint (none) -> SO16E
- U3: footprint ~ -> TSSOP16
- U5: footprint ~ -> SO14E
- U6: footprint ~ -> SO16E
- U7: footprint (none) -> SO16W
- U8: footprint ~ -> SO16W

Commit message: the TI TPS2095D datasheet suggests "shield shorted" should be inverted
Connections:
- net labels added: ~SHIELD_SHORTED~
- net labels removed: SHIELD_SHORTED

Commit message: renumber pogo-points to have same Px as main board test points
Parts:
- renumbered P20 to P1, P46 to P11, P47 to P12, P48 to P13, P49 to P14, P50 to P15, P51 to P16, P52 to P17, P53 to P18, P1 to P19, P21 to P2, P4 to P23, P5 to P24, P6 to P25, P7 to P26, P8 to P27, P9 to P28, P10 to P29, P22 to P3, P11 to P30, P12 to P31, P13 to P32, P14 to P33, P15 to P34, P16 to P35, P17 to P36, P18 to P37, P19 to P38, P29 to P39, P23 to P4, P30 to P40, P31 to P41, P32 to P42, P33 to P43, P34 to P44, P35 to P45, P36 to P46, P37 to P47, P38 to P48, P39 to P49, P24 to P5, P40 to P50, P41 to P51, P42 to P52, P43 to P53, P44 to P54, P45 to P55, P2 to P56, P3 to P57, P25 to P6, P26 to P7, P27 to P8, P28 to P9

Commit message: checkpoint tesh-harness pcb, components separated
Parts:
- P19: footprint arduino_shield -> arduino_shield_with_holes
Changed lines of the file:
@@
 F 0 "P19" H 4700 19000 60  0000 C CNN
 F 1 "ARDUINO_SHIELD" H 4700 18800 60  0000 C CNN
-F 2 "arduino_shield" H 4700 18900 60  0001 C CNN
+F 2 "arduino_shield_with_holes" H 4700 18900 60  0001 C CNN
 F 3 "" H 4700 18800 60  0001 C CNN
 	1    4700 18800

Commit message: re-order signal ladder for easier physical layout
Changed lines of the file:
@@
 	0    -1   -1   0
 $EndComp
-Text Label 7400 2650 2    60   ~ 0
+Text Label 4100 2800 0    60   ~ 0
 IN8P_LADDER
-Text Label 3900 2800 0    60   ~ 0
+Text Label 7600 2650 2    60   ~ 0
 IN8N_LADDER
 $Comp
@@
 	0    -1   -1   0
 $EndComp
-Text Label 7400 2950 2    60   ~ 0
+Text Label 4100 3100 0    60   ~ 0
 IN7P_LADDER
-Text Label 3900 3100 0    60   ~ 0
+Text Label 7600 2950 2    60   ~ 0
 IN7N_LADDER
 $Comp
@@
 	0    -1   -1   0
 $EndComp
-Text Label 7400 3250 2    60   ~ 0
+Text Label 4100 3400 0    60   ~ 0
 IN6P_LADDER
-Text Label 3900 3400 0    60   ~ 0
+Text Label 7600 3250 2    60   ~ 0
 IN6N_LADDER
 $Comp
@@
 	0    -1   -1   0
 $EndComp
-Text Label 7400 3550 2    60   ~ 0
+Text Label 4100 3700 0    60   ~ 0
 IN5P_LADDER
-Text Label 3900 3700 0    60   ~ 0
+Text Label 7600 3550 2    60   ~ 0
 IN5N_LADDER
 $Comp
@@
 	0    -1   -1   0
 $EndComp
-Text Label 7400 3850 2    60   ~ 0
+Text Label 4100 4000 0    60   ~ 0
 IN4P_LADDER
-Text Label 3900 4000 0    60   ~ 0
+Text Label 7600 3850 2    60   ~ 0
 IN4N_LADDER
 $Comp
@@
 	0    -1   -1   0
 $EndComp
-Text Label 7400 4150 2    60   ~ 0
+Text Label 4100 4300 0    60   ~ 0
 IN3P_LADDER
-Text Label 3900 4300 0    60   ~ 0
+Text Label 7600 4150 2    60   ~ 0
 IN3N_LADDER
 $Comp
@@
 	0    -1   -1   0
 $EndComp
-Text Label 7400 4450 2    60   ~ 0
+Text Label 4100 4600 0    60   ~ 0
 IN2P_LADDER
-Text Label 3900 4600 0    60   ~ 0
+Text Label 7600 4450 2    60   ~ 0
 IN2N_LADDER
 $Comp
@@
 	0    -1   -1   0
 $EndComp
-Text Label 7400 4750 2    60   ~ 0
+Text Label 4100 4900 0    60   ~ 0
 IN1P_LADDER
-Text Label 3900 4900 0    60   ~ 0
+Text Label 7600 4750 2    60   ~ 0
 IN1N_LADDER
 $Comp
@@
 	6400 6200 10250 6200
 Wire Wire Line
-	6000 2650 7400 2650
+	5500 2800 4100 2800
 Wire Wire Line
 	6100 2650 6100 2800
@@
 	6100 2800 6000 2800
 Wire Wire Line
-	3900 2800 5500 2800
+	7600 2650 6000 2650
 Wire Wire Line
 	5400 2800 5400 2950
@@
 Connection ~ 5400 2800
 Wire Wire Line
-	6000 2950 7400 2950
+	5500 3100 4100 3100
 Wire Wire Line
 	6100 2950 6100 3100
@@
 	6100 3100 6000 3100
 Wire Wire Line
-	3900 3100 5500 3100
+	7600 2950 6000 2950
 Wire Wire Line
 	5400 3100 5400 3250
@@
 Connection ~ 5400 3100
 Wire Wire Line
-	6000 3250 7400 3250
+	5500 3400 4100 3400
 Wire Wire Line
 	6100 3250 6100 3400
@@
 	6100 3400 6000 3400
 Wire Wire Line
-	3900 3400 5500 3400
+	7600 3250 6000 3250
 Wire Wire Line
 	5400 3400 5400 3550
@@
 Connection ~ 5400 3400
 Wire Wire Line
-	6000 3550 7400 3550
+	5500 3700 4100 3700
 Wire Wire Line
 	6100 3550 6100 3700
@@
 	6100 3700 6000 3700
 Wire Wire Line
-	3900 3700 5500 3700
+	7600 3550 6000 3550
 Wire Wire Line
 	5400 3700 5400 3850
@@
 Connection ~ 5400 3700
 Wire Wire Line
-	6000 3850 7400 3850
+	5500 4000 4100 4000
 Wire Wire Line
 	6100 3850 6100 4000
@@
 	6100 4000 6000 4000
 Wire Wire Line
-	3900 4000 5500 4000
+	7600 3850 6000 3850
 Wire Wire Line
 	5400 4000 5400 4150
@@
 Connection ~ 5400 4000
 Wire Wire Line
-	6000 4150 7400 4150
+	5500 4300 4100 4300
 Wire Wire Line
 	6100 4150 6100 4300
@@
 	6100 4300 6000 4300
 Wire Wire Line
-	3900 4300 5500 4300
+	7600 4150 6000 4150
 Wire Wire Line
 	5400 4300 5400 4450
@@
 Connection ~ 5400 4300
 Wire Wire Line
-	6000 4450 7400 4450
+	5500 4600 4100 4600
 Wire Wire Line
 	6100 4450 6100 4600
@@
 	6100 4600 6000 4600
 Wire Wire Line
-	3900 4600 5500 4600
+	7600 4450 6000 4450
 Wire Wire Line
 	5400 4600 5400 4750
@@
 Connection ~ 5400 4600
 Wire Wire Line
-	6000 4750 7400 4750
+	5500 4900 4100 4900
 Wire Wire Line
 	6100 4750 6100 4900
@@
 	6100 4900 6000 4900
 Wire Wire Line
-	3900 4900 5500 4900
+	7600 4750 6000 4750
 Wire Wire Line
 	5400 4900 5400 5050
@@
 	11700 3000 10400 3000
 Wire Wire Line
+	11700 3200 10400 3200
+Wire Wire Line
 	11700 3100 10400 3100
 Wire Wire Line
-	11700 3200 10400 3200
+	11700 3400 10400 3400
 Wire Wire Line
 	11700 3300 10400 3300
 Wire Wire Line
-	11700 3400 10400 3400
+	11700 3600 10400 3600
 Wire Wire Line
 	11700 3500 10400 3500
 Wire Wire Line
-	11700 3600 10400 3600
+	11700 3800 10400 3800
 Wire Wire Line
 	11700 3700 10400 3700
 Wire Wire Line
-	11700 3800 10400 3800
+	11700 4000 10400 4000
 Wire Wire Line
 	11700 3900 10400 3900
 Wire Wire Line
-	11700 4000 10400 4000
+	11700 4200 10400 4200
 Wire Wire Line
 	11700 4100 10400 4100
 Wire Wire Line
-	11700 4200 10400 4200
+	11700 4400 10400 4400
 Wire Wire Line
 	11700 4300 10400 4300
 Wire Wire Line
-	11700 4400 10400 4400
+	11700 4600 10400 4600
 Wire Wire Line
 	11700 4500 10400 4500
 Wire Wire Line
-	11700 4600 10400 4600
-Wire Wire Line
 	11700 2700 10400 2700
+Text Label 10400 4500 0    60   ~ 0
+IN1N_LADDER
 Text Label 10400 4600 0    60   ~ 0
-IN1N_LADDER
-Text Label 10400 4500 0    60   ~ 0
 IN1P_LADDER
+Text Label 10400 4300 0    60   ~ 0
+IN2N_LADDER
 Text Label 10400 4400 0    60   ~ 0
-IN2N_LADDER
-Text Label 10400 4300 0    60   ~ 0
 IN2P_LADDER
+Text Label 10400 4100 0    60   ~ 0
+IN3N_LADDER
 Text Label 10400 4200 0    60   ~ 0
-IN3N_LADDER
-Text Label 10400 4100 0    60   ~ 0
 IN3P_LADDER
+Text Label 10400 3900 0    60   ~ 0
+IN4N_LADDER
 Text Label 10400 4000 0    60   ~ 0
-IN4N_LADDER
-Text Label 10400 3900 0    60   ~ 0
 IN4P_LADDER
+Text Label 10400 3700 0    60   ~ 0
+IN5N_LADDER
 Text Label 10400 3800 0    60   ~ 0
-IN5N_LADDER
-Text Label 10400 3700 0    60   ~ 0
 IN5P_LADDER
+Text Label 10400 3500 0    60   ~ 0
+IN6N_LADDER
 Text Label 10400 3600 0    60   ~ 0
-IN6N_LADDER
-Text Label 10400 3500 0    60   ~ 0
 IN6P_LADDER
+Text Label 10400 3300 0    60   ~ 0
+IN7N_LADDER
 Text Label 10400 3400 0    60   ~ 0
-IN7N_LADDER
-Text Label 10400 3300 0    60   ~ 0
 IN7P_LADDER
+Text Label 10400 3100 0    60   ~ 0
+IN8N_LADDER
 Text Label 10400 3200 0    60   ~ 0
-IN8N_LADDER
-Text Label 10400 3100 0    60   ~ 0
 IN8P_LADDER
 Text Label 10400 2900 0    60   ~ 0
@@
 	12500 3000 13800 3000
 Wire Wire Line
+	12500 3200 13800 3200
+Wire Wire Line
 	12500 3100 13800 3100
 Wire Wire Line
-	12500 3200 13800 3200
+	12500 3400 13800 3400
 Wire Wire Line
 	12500 3300 13800 3300
 Wire Wire Line
-	12500 3400 13800 3400
+	12500 3600 13800 3600
 Wire Wire Line
 	12500 3500 13800 3500
 Wire Wire Line
-	12500 3600 13800 3600
+	12500 3800 13800 3800
 Wire Wire Line
 	12500 3700 13800 3700
 Wire Wire Line
-	12500 3800 13800 3800
+	12500 4000 13800 4000
 Wire Wire Line
 	12500 3900 13800 3900
 Wire Wire Line
-	12500 4000 13800 4000
+	12500 4200 13800 4200
 Wire Wire Line
 	12500 4100 13800 4100
 Wire Wire Line
-	12500 4200 13800 4200
+	12500 4400 13800 4400
 Wire Wire Line
 	12500 4300 13800 4300
 Wire Wire Line
-	12500 4400 13800 4400
+	12500 4600 13800 4600
 Wire Wire Line
 	12500 4500 13800 4500
-Wire Wire Line
-	12500 4600 13800 4600
+Text Label 13800 4500 2    60   ~ 0
+IN1N
 Text Label 13800 4600 2    60   ~ 0
-IN1N
-Text Label 13800 4500 2    60   ~ 0
 IN1P
+Text Label 13800 4300 2    60   ~ 0
+IN2N
 Text Label 13800 4400 2    60   ~ 0
-IN2N
-Text Label 13800 4300 2    60   ~ 0
 IN2P
+Text Label 13800 4100 2    60   ~ 0
+IN3N
 Text Label 13800 4200 2    60   ~ 0
-IN3N
-Text Label 13800 4100 2    60   ~ 0
 IN3P
+Text Label 13800 3900 2    60   ~ 0
+IN4N
 Text Label 13800 4000 2    60   ~ 0
-IN4N
-Text Label 13800 3900 2    60   ~ 0
 IN4P
+Text Label 13800 3700 2    60   ~ 0
+IN5N
 Text Label 13800 3800 2    60   ~ 0
-IN5N
-Text Label 13800 3700 2    60   ~ 0
 IN5P
+Text Label 13800 3500 2    60   ~ 0
+IN6N
 Text Label 13800 3600 2    60   ~ 0
-IN6N
-Text Label 13800 3500 2    60   ~ 0
 IN6P
+Text Label 13800 3300 2    60   ~ 0
+IN7N
 Text Label 13800 3400 2    60   ~ 0
-IN7N
-Text Label 13800 3300 2    60   ~ 0
 IN7P
+Text Label 13800 3100 2    60   ~ 0
+IN8N
 Text Label 13800 3200 2    60   ~ 0
-IN8N
-Text Label 13800 3100 2    60   ~ 0
 IN8P
 Text Label 13800 3000 2    60   ~ 0

Commit message: untangle the rats nest some
Parts:
- removed R45, R46, R47, R48, R49, R50: 47, SM0603, symbol R
Connections:
- net labels added: 3.3V_BOGUS_ISO_DATA, A1, A2, A3, A4, LED1, LED2, LED3, MIDDLE_CARRY, VCC_DATA, VDD1, VISO_BOGUS_ISO_PRE
- wire segments 454 -> 450
Other:
- moved on the sheet: D1, D2, D3

Commit message: power chips on isolated side of test harness from the board under test
Parts:
- removed C13, C14, C7, C8: 100nF, SM0603, symbol C
- removed C15, C16, C5, C6: 10uF, SM0805, symbol C
- removed L2, L5: MH2029-221Y, SM0805, symbol INDUCTOR
- removed U7: ADUM6000, SO16W, symbol ADUM6000
Connections:
- net labels removed: VDD1, VISO_BOGUS_ISO_PRE
- wire segments 450 -> 395
- no-connect marks 19 -> 17
Other:
- note removed: "Bogus Power Isolation"
- note removed: "Note that bypass capacitors should be\nvery close to the chip and the grounds\nconnectted together with a very low\nimpedence connection\n(wide traces, large vias)"
- note removed: "bypass capacitors"
