File: kicad-files/OpenHardwareExG_Shield_Test_Board.sch (KiCad schematic (older format))
At the start: 119 parts, among them P1 CONN_1, P11 CONN_1, P12 CONN_1, P13 CONN_1, P14 CONN_1, P15 CONN_1, P16 CONN_1, P17 CONN_1, P18 CONN_1, P19 ARDUINO_SHIELD, P2 CONN_1, P23 CONN_1, P24 CONN_1, P25 CONN_1, P26 CONN_1, P27 CONN_1, P28 CONN_1, P29 CONN_1, P3 CONN_1, P30 CONN_1, P31 CONN_1, P32 CONN_1, P33 CONN_1, P34 CONN_1, P35 CONN_1, P36 CONN_1, P37 CONN_1, P38 CONN_1, P39 CONN_1, P4 CONN_1, P40 CONN_1, P41 CONN_1, P42 CONN_1, P43 CONN_1, P44 CONN_1, P45 CONN_1, P46 CONN_1, P47 CONN_1, P48 CONN_1, P49 CONN_1, P5 CONN_1, P50 CONN_1, P51 CONN_1, P52 CONN_1, P53 CONN_1, P54 CONN_1, P55 CONN_1, P56 CONN_3X2, P57 CONN_20X2, P6 CONN_1, P7 CONN_1, P8 CONN_1, P9 CONN_1, SW1 SW_PUSH, U1 74HC165, U2 74HC165, U3 74HC595PWR, U4 74HC165, U5 74LS125, U6 TPS2095D, U8 SI8661

Commit message: routing of test harness half done
Parts:
- added C5: 10uF, SM0805, symbol C
- added C6, C7, C8: 100nF, SM0603, symbol C
Connections:
- net labels removed: DGND_BOGUS_ISO
- wire segments 395 -> 405
Changed lines of the file:
@@
 3.3V_BOGUS_ISO
 Text Label 850  19500 0    60   ~ 0
-DGND_BOGUS_ISO
+GND_BOGUS_ISO
 $Comp
 L R R1
@@
 $EndComp
 Text Label 2150 17450 2    60   ~ 0
-DGND_BOGUS_ISO
+GND_BOGUS_ISO
 $Comp
 L R R8
@@
 3.3V_BOGUS_ISO
 Text Label 12700 13800 0    60   ~ 0
-DGND_BOGUS_ISO
+GND_BOGUS_ISO
 $Comp
 L CONN_1 P29
@@
 	20450 9650 20450 9800
 Connection ~ 20450 9800
+Text Notes 21850 18650 1    45   ~ 0
+SHIFT
+Text Notes 21500 18650 1    45   ~ 0
+SHIFT
+Text Notes 21150 18650 1    45   ~ 0
+Buffer
+$Comp
+L C C8
+U 1 1 550458EB
+P 21850 18950
+F 0 "C8" H 21900 19050 50  0000 L CNN
+F 1 "100nF" H 21900 18850 50  0000 L CNN
+F 2 "SM0603" H 21900 18950 50  0001 C CNN
+F 3 "" H 21850 18950 60  0001 C CNN
+	1    21850 18950
+	1    0    0    -1
+$EndComp
+$Comp
+L C C7
+U 1 1 550458F1
+P 21500 18950
+F 0 "C7" H 21550 19050 50  0000 L CNN
+F 1 "100nF" H 21550 18850 50  0000 L CNN
+F 2 "SM0603" H 21550 18950 50  0001 C CNN
+F 3 "" H 21500 18950 60  0001 C CNN
+	1    21500 18950
+	1    0    0    -1
+$EndComp
+$Comp
+L C C5
+U 1 1 550458F7
+P 20800 18950
+F 0 "C5" H 20850 19050 50  0000 L CNN
+F 1 "10uF" H 20850 18850 50  0000 L CNN
+F 2 "SM0805" H 20850 18950 50  0001 C CNN
+F 3 "" H 20800 18950 60  0001 C CNN
+	1    20800 18950
+	1    0    0    -1
+$EndComp
+$Comp
+L C C6
+U 1 1 550458FD
+P 21150 18950
+F 0 "C6" H 21200 19050 50  0000 L CNN
+F 1 "100nF" H 21200 18850 50  0000 L CNN
+F 2 "SM0603" H 21200 18950 50  0001 C CNN
+F 3 "" H 21150 18950 60  0001 C CNN
+	1    21150 18950
+	1    0    0    -1
+$EndComp
+Connection ~ 20800 18700
+Wire Wire Line
+	20800 18700 20800 18750
+Connection ~ 21500 18700
+Wire Wire Line
+	21500 18700 21500 18750
+Wire Wire Line
+	21850 19200 21850 19150
+Connection ~ 21150 19200
+Wire Wire Line
+	21150 19200 21150 19150
+Wire Wire Line
+	20000 19200 21850 19200
+Wire Wire Line
+	20800 19200 20800 19150
+Connection ~ 20800 19200
+Wire Wire Line
+	21500 19200 21500 19150
+Connection ~ 21500 19200
+Wire Wire Line
+	21850 18700 21850 18750
+Wire Wire Line
+	21150 18700 21150 18750
+Connection ~ 21150 18700
+Wire Wire Line
+	20000 18700 21850 18700
+Text Label 20000 18700 0    60   ~ 0
+ARDUINO_VCC
+Text Label 20000 19200 0    60   ~ 0
+ARDUINO_GND
 $EndSCHEMATC

Commit message: finish initial routing of the test board
Connections:
- net labels added: UNUSED
- wire segments 405 -> 407
Changed lines of the file:
@@
 Sheet 1 1
 Title ""
-Date "14 mar 2015"
+Date "21 mar 2015"
 Rev ""
 Comp ""
@@
 Text Label 10250 7600 2    60   ~ 0
 ADS129x_CLK_BOGUS_ISO
-Text Label 17350 20200 2    60   ~ 0
-3.3V_BOGUS_ISO
-Text Label 10250 6100 2    60   ~ 0
-3.3V_BOGUS_ISO
 Text Label 10250 6200 2    60   ~ 0
 SHIFT_EXT_CARRY_BOGUS_ISO
-Text Label 10250 7500 2    60   ~ 0
-3.3V_BOGUS_ISO
 $Comp
 L R R17
@@
 	1    0    0    -1
 $EndComp
-$Comp
-L GND #PWR022
-U 1 1 544BD63D
-P 15150 21000
-F 0 "#PWR022" H 15150 21000 30  0001 C CNN
-F 1 "GND" H 15150 20930 30  0001 C CNN
-F 2 "" H 15150 21000 60  0000 C CNN
-F 3 "" H 15150 21000 60  0000 C CNN
-	1    15150 21000
-	1    0    0    -1
-$EndComp
 NoConn ~ 20600 14400
 Text Label 3150 18050 2    60   ~ 0
@@
 Text Label 17550 18500 2    60   ~ 0
 ARDUINO_VCC
-Text Label 10250 5800 2    60   ~ 0
-3.3V_BOGUS_ISO
 Text Label 10250 5700 2    60   ~ 0
 GND_BOGUS_ISO
@@
 	6400 7300 6900 7300
 Wire Wire Line
-	6400 7500 10250 7500
+	10850 7500 6400 7500
 Wire Wire Line
 	6400 7600 10250 7600
@@
 	6400 6000 10250 6000
 Wire Wire Line
-	6400 6100 10250 6100
+	10850 6100 6400 6100
 Wire Wire Line
 	6400 6200 10250 6200
@@
 	15000 18900 13800 18900
 Wire Wire Line
-	6400 5800 10250 5800
+	6400 5800 10850 5800
 Wire Wire Line
 	6400 5700 10250 5700
@@
 Text Label 20000 19200 0    60   ~ 0
 ARDUINO_GND
+Text Label 17350 20200 2    60   ~ 0
+ARDUINO_VCC
+Wire Wire Line
+	10850 5450 10850 7500
+Connection ~ 10850 5800
+$Comp
+L VCC #PWR029
+U 1 1 550D64DE
+P 10850 5450
+F 0 "#PWR029" H 10850 5550 30  0001 C CNN
+F 1 "VCC" H 10850 5550 30  0000 C CNN
+F 2 "" H 10850 5450 60  0000 C CNN
+F 3 "" H 10850 5450 60  0000 C CNN
+	1    10850 5450
+	1    0    0    -1
+$EndComp
+Connection ~ 10850 6100
+Text Label 10250 5800 2    60   ~ 0
+UNUSED
+Text Label 10250 7500 2    60   ~ 0
+UNUSED
+Text Label 10250 6100 2    60   ~ 0
+UNUSED
+Text Label 17350 21000 2    60   ~ 0
+ARDUINO_GND
+Wire Wire Line
+	15150 21000 17350 21000
 $EndSCHEMATC

Commit message: add notes about connecting test points for next rev
Parts:
- C1, C10, C11, C12, C2, C3, C4, C5, C6, C7, C8, C9: symbol C -> C-RESCUE-OpenHardwareExG_Shield_Test_Board
- D1, D2, D3: symbol LED -> LED-RESCUE-OpenHardwareExG_Shield_Test_Board
- R1, R10, R11, R12, R13, R14, R15, R16, R17, R18, R19, R2, R20, R21, R22, R23, R24, R25, R26, R27, R28, R29, R3, R30, R31, R32, R33, R34, R35, R36, R37, R38, R39, R4, R40, R41, R42, R43, R44, R5, R6, R7, R8, R9: symbol R -> R-RESCUE-OpenHardwareExG_Shield_Test_Board
- U8: symbol SI8661 -> Si8661
