File: kicad-files/OpenHardwareExG_Shield_Test_Board.kicad_pcb (KiCad board)
At the start: 4 copper layers, 147.3 x 81.3 mm, 137 parts, among them P1 CONN_1, P11 CONN_1, P12 CONN_1, P13 CONN_1, P14 CONN_1, P15 CONN_1, P16 CONN_1, P17 CONN_1, P18 CONN_1, P19 ARDUINO_SHIELD, P2 CONN_1, P23 CONN_1, P24 CONN_1, P25 CONN_1, P26 CONN_1, P27 CONN_1, P28 CONN_1, P29 CONN_1, P3 CONN_1, P30 CONN_1, P31 CONN_1, P32 CONN_1, P33 CONN_1, P34 CONN_1, P35 CONN_1, P36 CONN_1, P37 CONN_1, P38 CONN_1, P39 CONN_1, P4 CONN_1, P40 CONN_1, P41 CONN_1, P42 CONN_1, P43 CONN_1, P44 CONN_1, P45 CONN_1, P46 CONN_1, P47 CONN_1, P48 CONN_1, P49 CONN_1, P5 CONN_1, P50 CONN_1, P51 CONN_1, P52 CONN_1, P53 CONN_1, P54 CONN_1, P55 CONN_1, P56 CONN_3X2, P57 CONN_20X2, P6 CONN_1, P7 CONN_1, P8 CONN_1, P9 CONN_1, SW1 SW_PUSH, U1 74HC165, U2 74HC165, U3 74HC595PWR, U4 74HC165, U5 74LS125, U6 TPS2095D, U8 SI8661

Commit message: improve routing of ground and power; improve planes on BOGUS_ISO side
Routing:
- net VCC: track 18.8 -> 239.9 mm, vias 2 -> 26
- net GND: track 130.4 -> 322.9 mm, vias 30 -> 47
- net /3.3V_BOGUS_ISO: track 134.2 -> 156.9 mm, vias 6 -> 10
- net (no net): track 3.11 -> 0.00 mm, vias 2 -> 0
- net /SHIFT_SH_~LD~_BOGUS_ISO: track 114.1 -> 111.2 mm
- net /MASTER_BOGUS_ISO: track 56.7 -> 54.0 mm
- net /ADS129x_CLK_BOGUS_ISO: track 36.4 -> 38.8 mm
- net /SHIFT_CARRY_BOGUS_ISO: track 66.0 -> 67.5 mm
- net /ADS129x_DOUT_BOGUS_ISO: track 42.5 -> 41.3 mm
- net /SHIFT_EXT_CARRY_BOGUS_ISO: track 69.4 -> 70.5 mm
- net /BIASINV: track 21.2 -> 22.3 mm
- net /MIDDLE_CARRY: track 20.3 -> 21.2 mm
- net /SIGNAL_B_BOGUS_ISO: track 50.2 -> 50.8 mm
- net /SHIFT_CLK_BOGUS_ISO: track 102.2 -> 102.9 mm
- net /ADS129x_GPIO1_BOGUS_ISO: track 27.7 -> 28.4 mm
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
Commit message: improved routing and planes on test board
Routing:
- net GNDPWR: track 43.8 -> 221.4 mm, vias 19 -> 54
- net /ARDUINO_VCC: track 3.39 -> 178.9 mm, vias 0 -> 24
- net VCC: track 239.9 -> 249.9 mm
- net /SHIFT_OUT_RCLK: track 13.5 -> 15.0 mm, vias 0 -> 2
- net /SHIFT_CARRY: track 54.0 -> 55.3 mm
- net /~SHIELD_SHORTED~: track 65.5 -> 64.4 mm, vias 4 -> 3
- net /GO_BUTTON: track 31.8 -> 32.9 mm
- net /ENABLE_SHIELD: track 50.9 -> 51.8 mm
- net /ADS129x_~DRDY~: track 29.2 -> 28.3 mm
- net /SHIFT_OUT_SRCLK: track 16.0 -> 16.7 mm, vias 0 -> 2
- net /MASTER_AND_MASTER_CS: track 12.7 -> 13.5 mm
- net +5V: track 175.3 -> 174.6 mm
- net /SHIFT_OUT_~SRCLR~: track 18.0 -> 18.7 mm, vias 0 -> 2
- net /SHIFT_OUT: track 14.5 -> 13.8 mm, vias 0 -> 1
- net /SIGNAL_B: track 44.8 -> 45.5 mm
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