File: OpenHardwareExG_Shield_Test_Harness/kicad-files/OpenHardwareExG_Shield_Test_Board.sch (KiCad schematic (older format))
At the start: 123 parts, among them P1 CONN_1, P11 CONN_1, P12 CONN_1, P13 CONN_1, P14 CONN_1, P15 CONN_1, P16 CONN_1, P17 CONN_1, P18 CONN_1, P19 ARDUINO_SHIELD, P2 CONN_1, P23 CONN_1, P24 CONN_1, P25 CONN_1, P26 CONN_1, P27 CONN_1, P28 CONN_1, P29 CONN_1, P3 CONN_1, P30 CONN_1, P31 CONN_1, P32 CONN_1, P33 CONN_1, P34 CONN_1, P35 CONN_1, P36 CONN_1, P37 CONN_1, P38 CONN_1, P39 CONN_1, P4 CONN_1, P40 CONN_1, P41 CONN_1, P42 CONN_1, P43 CONN_1, P44 CONN_1, P45 CONN_1, P46 CONN_1, P47 CONN_1, P48 CONN_1, P49 CONN_1, P5 CONN_1, P50 CONN_1, P51 CONN_1, P52 CONN_1, P53 CONN_1, P54 CONN_1, P55 CONN_1, P56 CONN_3X2, P57 CONN_20X2, P6 CONN_1, P7 CONN_1, P8 CONN_1, P9 CONN_1, SW1 SW_PUSH, U1 74HC165, U2 74HC165, U3 74HC595PWR, U4 74HC165, U5 74LS125, U6 TPS2095D, U8 SI8661

Commit message: adjust for new version of KiCAD, copy in lib from main project
Parts:
- C1, C10, C11, C12, C2, C3, C4, C5, C6, C7, C8, C9: symbol C-RESCUE-OpenHardwareExG_Shield_Test_Board -> C
- D1, D2, D3: symbol LED-RESCUE-OpenHardwareExG_Shield_Test_Board -> LED
- R1, R10, R11, R12, R13, R14, R15, R16, R17, R18, R19, R2, R20, R21, R22, R23, R24, R25, R26, R27, R28, R29, R3, R30, R31, R32, R33, R34, R35, R36, R37, R38, R39, R4, R40, R41, R42, R43, R44, R5, R6, R7, R8, R9: symbol R-RESCUE-OpenHardwareExG_Shield_Test_Board -> R
